Commit message: update maze.

File: envs/data/maze.urdf (robot description, URDF)
Before this commit: robot cube.urdf, 8 links, 7 joints
Links:
- link wall1: geometry collision box size=.01 .18 .05; visual box size=.01 .18 .05
- link wall2: geometry collision box size=.17 .01 .05; visual box size=.17 .01 .05
- link wall3: geometry collision box size=.01 .04 .05; visual box size=.01 .04 .05
- link wall4: geometry collision box size=.08 .01 .05; visual box size=.08 .01 .05
- link wall5: geometry collision box size=.01 .08 .05; visual box size=.01 .08 .05
- link wall6: geometry collision box size=.08 .01 .05; visual box size=.08 .01 .05
- link wall7: geometry collision box size=.01 .04 .05; visual box size=.01 .04 .05
- link wall8: geometry collision box size=.17 .01 .05; visual box size=.17 .01 .05
Joints:
- joint wall1_wall2_joint: origin xyz=.045 -.07 0 rpy=0 0 0 -> xyz=.09 -.085 0 rpy=0 0 0
- joint wall2_wall3_joint: origin xyz=.035 .015 0 rpy=0 0 0 -> xyz=.08 .025 0 rpy=0 0 0
- joint wall3_wall4_joint: origin xyz=-.015 .015 0 rpy=0 0 0 -> xyz=-.035 .025 0 rpy=0 0 0
- joint wall4_wall5_joint: origin xyz=-.025 .04 0 rpy=0 0 0 -> xyz=-.045 .035 0 rpy=0 0 0
- joint wall5_wall6_joint: origin xyz=.025 .040 0 rpy=0 0 0 -> xyz=.045 .035 0 rpy=0 0 0
- joint wall6_wall7_joint: origin xyz=.015 .015 0 rpy=0 0 0 -> xyz=.035 .025 0 rpy=0 0 0
- joint wall7_wall8_joint: origin xyz=-.035 .015 0 rpy=0 0 0 -> xyz=-.08 .025 0 rpy=0 0 0

File: envs/data/stick.urdf (robot description, URDF)
Before this commit: robot stick, 1 links, 0 joints
Links:
- link stick: geometry collision cylinder length=0.08 radius=0.004; visual cylinder length=0.08 radius=0.008
