Commit message: Update readme.

File: envs/data/maze2.urdf (robot description, URDF)
Before this commit: robot maze2.urdf, 8 links, 7 joints
Links:
- link wall1: geometry collision box size=.01 .34 .05; visual box size=.01 .34 .05
- link wall2: geometry collision box size=.17 .01 .05; visual box size=.17 .01 .05
- link wall5: geometry collision box size=.01 .24 .05; visual box size=.01 .24 .05
- link wall8: geometry collision box size=.17 .01 .05; visual box size=.17 .01 .05
Joints:
- joint wall1_wall2_joint: origin xyz=.09 -.085 0 rpy=0 0 0 -> xyz=.09 -.165 0 rpy=0 0 0
- joint wall4_wall5_joint: origin xyz=-.045 .035 0 rpy=0 0 0 -> xyz=-.045 .115 0 rpy=0 0 0
- joint wall5_wall6_joint: origin xyz=.045 .035 0 rpy=0 0 0 -> xyz=.045 .115 0 rpy=0 0 0
